File: hw/loop_antenna_amp/loop_antenna_amp.sch (KiCad schematic (older format))
At the start: 87 parts, among them J1 ANT1, J2 ANT2, J3 GND, J4 Coax (SMA), Q1 MMBT3904, Q2 MMBT3904, Q3 MMBT3904, Q4 MMBT3904, Q5 PZT3904, Q6 PZT3904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

Commit message: Loop antenna amp: simplify input protection
Parts:
- removed D5, D6: LL4148, Diode_SMD:D_MiniMELF, symbol Diode:1N4148W
- renumbered D7 to D5, D8 to D6, D9 to D7, D10 to D8
Connections:
- net at D2.1 (K), D3.2 (A): now also Q2.2 (E), T1.3 (SA), T2.3 (AC); no longer D4.1 (K)
- net at D2.2 (A), Q1.2 (E), T1.4 (SB)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: now also D3.1 (K)
- net at C4.1, C6.1, R4.1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: now also D4.1 (K)
Other:
- moved on the sheet: D2, D3, D4
Changed lines of the file:
@@
 L Device:D_Zener D4
 U 1 1 60C8EF37
-P 3250 3750
-F 0 "D4" V 3204 3670 50  0000 R CNN
-F 1 "BZV55-C4V7" V 3295 3670 50  0000 R CNN
-F 2 "Diode_SMD:D_MiniMELF" H 3250 3750 50  0001 C CNN
-F 3 "~" H 3250 3750 50  0001 C CNN
-	1    3250 3750
+P 3400 3750
+F 0 "D4" V 3354 3670 50  0000 R CNN
+F 1 "BZV55-C4V7" V 3445 3670 50  0000 R CNN
+F 2 "Diode_SMD:D_MiniMELF" H 3400 3750 50  0001 C CNN
+F 3 "~" H 3400 3750 50  0001 C CNN
+	1    3400 3750
 	0    1    1    0
 $EndComp
@@
 L power:GND #PWR07
 U 1 1 60C98F98
-P 3250 4000
-F 0 "#PWR07" H 3250 3750 50  0001 C CNN
-F 1 "GND" H 3255 3827 50  0000 C CNN
-F 2 "" H 3250 4000 50  0001 C CNN
-F 3 "" H 3250 4000 50  0001 C CNN
-	1    3250 4000
-	1    0    0    -1
-$EndComp
-Wire Wire Line
-	3250 3600 3250 2200
-Wire Wire Line
-	3250 3900 3250 4000
+P 3400 4000
+F 0 "#PWR07" H 3400 3750 50  0001 C CNN
+F 1 "GND" H 3405 3827 50  0000 C CNN
+F 2 "" H 3400 4000 50  0001 C CNN
+F 3 "" H 3400 4000 50  0001 C CNN
+	1    3400 4000
+	1    0    0    -1
+$EndComp
+Wire Wire Line
+	3400 3900 3400 4000
 $Comp
 L power:GND #PWR010
@@
 	1200 3000 1500 3000
 Wire Wire Line
-	3250 2200 3400 2200
-Connection ~ 3250 2200
-Wire Wire Line
 	4150 2400 4150 3000
 Wire Wire Line
@@
 Connection ~ 4150 3000
 Wire Wire Line
-	3400 3000 4150 3000
-Wire Wire Line
 	5050 3000 4150 3000
 Wire Wire Line
 	4150 1400 4150 2000
-Wire Wire Line
-	3400 1400 4150 1400
 Wire Wire Line
 	5050 1400 4150 1400
@@
 L Diode:1N4148W D2
 U 1 1 60C87CF8
-P 3100 1800
-F 0 "D2" V 3146 1880 50  0000 L CNN
-F 1 "LL4148" V 3055 1880 50  0000 L CNN
-F 2 "Diode_SMD:D_MiniMELF" H 3100 1625 50  0001 C CNN
-F 3 "https://www.vishay.com/docs/85748/1n4148w.pdf" H 3100 1800 50  0001 C CNN
-	1    3100 1800
+P 3100 2200
+F 0 "D2" V 3146 2279 50  0000 L CNN
+F 1 "LL4148" V 3055 2279 50  0000 L CNN
+F 2 "Diode_SMD:D_MiniMELF" H 3100 2025 50  0001 C CNN
+F 3 "https://www.vishay.com/docs/85748/1n4148w.pdf" H 3100 2200 50  0001 C CNN
+	1    3100 2200
 	0    -1   -1   0
-$EndComp
-$Comp
-L Diode:1N4148W D5
-U 1 1 60C89AB8
-P 3400 1800
-F 0 "D5" V 3354 1880 50  0000 L CNN
-F 1 "LL4148" V 3445 1880 50  0000 L CNN
-F 2 "Diode_SMD:D_MiniMELF" H 3400 1625 50  0001 C CNN
-F 3 "https://www.vishay.com/docs/85748/1n4148w.pdf" H 3400 1800 50  0001 C CNN
-	1    3400 1800
-	0    1    1    0
 $EndComp
 Wire Wire Line
@@
 	-1   0    0    1
 $EndComp
-Connection ~ 3400 1400
-Connection ~ 3400 3000
 $Comp
 L local_syms:Transformer_1PS_2S_ferrite T2
@@
 	1    0    0    -1
 $EndComp
-Wire Wire Line
-	3400 2200 3400 2450
-Connection ~ 3400 2200
-Wire Wire Line
-	3100 2200 3100 2450
-Connection ~ 3100 2200
-Wire Wire Line
-	3100 2200 3250 2200
 Connection ~ 3100 3000
-Wire Wire Line
-	3100 2750 3100 3000
-Wire Wire Line
-	3100 1400 3400 1400
 Connection ~ 3100 1400
-Wire Wire Line
-	3100 1650 3100 1400
-Wire Wire Line
-	3400 1400 3400 1650
-Wire Wire Line
-	3400 3000 3100 3000
-Wire Wire Line
-	3400 2750 3400 3000
-Wire Wire Line
-	3400 1950 3400 2200
-Wire Wire Line
-	3100 1950 3100 2200
 $Comp
 L Diode:1N4148W D3
 U 1 1 60C8B51B
-P 3100 2600
-F 0 "D3" V 3146 2680 50  0000 L CNN
-F 1 "LL4148" V 3055 2680 50  0000 L CNN
-F 2 "Diode_SMD:D_MiniMELF" H 3100 2425 50  0001 C CNN
-F 3 "https://www.vishay.com/docs/85748/1n4148w.pdf" H 3100 2600 50  0001 C CNN
-	1    3100 2600
-	0    -1   -1   0
-$EndComp
-$Comp
-L Diode:1N4148W D6
-U 1 1 60C8A5AB
-P 3400 2600
-F 0 "D6" V 3354 2680 50  0000 L CNN
-F 1 "LL4148" V 3445 2680 50  0000 L CNN
-F 2 "Diode_SMD:D_MiniMELF" H 3400 2425 50  0001 C CNN
-F 3 "https://www.vishay.com/docs/85748/1n4148w.pdf" H 3400 2600 50  0001 C CNN
-	1    3400 2600
+P 3400 2200
+F 0 "D3" V 3354 2280 50  0000 L CNN
+F 1 "LL4148" V 3445 2280 50  0000 L CNN
+F 2 "Diode_SMD:D_MiniMELF" H 3400 2025 50  0001 C CNN
+F 3 "https://www.vishay.com/docs/85748/1n4148w.pdf" H 3400 2200 50  0001 C CNN
+	1    3400 2200
 	0    1    1    0
 $EndComp
@@
 	4850 2250 4850 4750
 $Comp
-L Diode:1N4148W D8
+L Diode:1N4148W D6
 U 1 1 60CC2F1F
 P 5250 2450
-F 0 "D8" V 5300 2650 50  0000 R CNN
-F 1 "LL4148" V 5200 2900 50  0000 R CNN
+F 0 "D6" V 5300 2650 50  0000 R CNN
+F 1 "LL4148" V 5200 2800 50  0000 R CNN
 F 2 "Diode_SMD:D_MiniMELF" H 5250 2275 50  0001 C CNN
 F 3 "https://www.vishay.com/docs/85748/1n4148w.pdf" H 5250 2450 50  0001 C CNN
@@
 	5250 2650 5250 2700
 $Comp
-L Diode:1N4148W D7
+L Diode:1N4148W D5
 U 1 1 60CC5B68
 P 5250 1950
-F 0 "D7" V 5200 2150 50  0000 R CNN
-F 1 "LL4148" V 5300 2400 50  0000 R CNN
+F 0 "D5" V 5204 2029 50  0000 L CNN
+F 1 "LL4148" V 5295 2029 50  0000 L CNN
 F 2 "Diode_SMD:D_MiniMELF" H 5250 1775 50  0001 C CNN
 F 3 "https://www.vishay.com/docs/85748/1n4148w.pdf" H 5250 1950 50  0001 C CNN
@@
 Connection ~ 4650 3500
 $Comp
-L Diode:1N4148W D10
+L Diode:1N4148W D8
 U 1 1 611B538C
 P 7550 3500
-F 0 "D10" H 7550 3283 50  0000 C CNN
+F 0 "D8" H 7550 3283 50  0000 C CNN
 F 1 "LL4148" H 7550 3374 50  0000 C CNN
 F 2 "Diode_SMD:D_MiniMELF" H 7550 3325 50  0001 C CNN
@@
 	7150 3200 7150 3250
 $Comp
-L Diode:1N4148W D9
+L Diode:1N4148W D7
 U 1 1 611C9E8F
 P 7550 900
-F 0 "D9" H 7550 683 50  0000 C CNN
+F 0 "D7" H 7550 683 50  0000 C CNN
 F 1 "LL4148" H 7550 774 50  0000 C CNN
 F 2 "Diode_SMD:D_MiniMELF" H 7550 725 50  0001 C CNN
@@
 Wire Wire Line
 	9600 3050 10000 3050
+Wire Wire Line
+	3400 3600 3400 3500
+Wire Wire Line
+	3400 3500 3850 3500
+Wire Wire Line
+	3100 3000 3400 3000
+Wire Wire Line
+	3100 1400 3400 1400
+Wire Wire Line
+	3100 1400 3100 2050
+Wire Wire Line
+	3400 2050 3400 1400
+Connection ~ 3400 1400
+Wire Wire Line
+	3400 1400 4150 1400
+Wire Wire Line
+	3400 2350 3400 3000
+Connection ~ 3400 3000
+Wire Wire Line
+	3400 3000 4150 3000
+Wire Wire Line
+	3100 2350 3100 3000
 $EndSCHEMATC

Commit message: Loop antenna amp: fix antenna connector polarity markings
Parts:
- J1: value ANT1 -> ANT+
- J2: value ANT2 -> ANT-
Changed lines of the file:
@@
 P 1000 3000
 F 0 "J2" H 918 2775 50  0000 C CNN
-F 1 "ANT2" H 918 2866 50  0000 C CNN
+F 1 "ANT-" H 918 2866 50  0000 C CNN
 F 2 "local_footprints:Keystone_7771_ScrewTerminal" H 1000 3000 50  0001 C CNN
 F 3 "~" H 1000 3000 50  0001 C CNN
@@
 P 1000 1400
 F 0 "J1" H 918 1175 50  0000 C CNN
-F 1 "ANT1" H 918 1266 50  0000 C CNN
+F 1 "ANT+" H 918 1266 50  0000 C CNN
 F 2 "local_footprints:Keystone_7771_ScrewTerminal" H 1000 1400 50  0001 C CNN
 F 3 "~" H 1000 1400 50  0001 C CNN

Commit message: Loop antenna amp: document actual transformer design
Other:
- note added: "Transformers T1, T2, T3:\nsee TRANSFORMERS.md file for instructions"
- note removed: "Transformer T1:\n Fair-Rite 5943004901 toroid\n 5 turns of RG174\n\nTransformer T2:\n Fair-Rite 2843000202 core (BN-43-202)\n 0.3mm magnetic copper wire\n 1-2: 1 turn\n 2-3: 1 turn\n 4-5: 8 turns\n 6-7: 8 turns\n\nTransformer T3:\n Fair-Rite 2843000202 core (BN-43-202)\n 10 turns of twisted pair made from\n 0.3mm magnetic copper wire\n"
Changed lines of the file:
@@
 Title "Lomiloop antenna amplifier"
 Date "2021-06-14"
-Rev ""
+Rev "1"
 Comp "Roman Dobrodii"
 Comment1 "Licensed under Solderpad Hardware License v2.1"
@@
 Wire Wire Line
 	6500 7050 6500 7150
-Text Notes 1000 5400 0    50   ~ 0
-Transformer T1:\n  Fair-Rite 5943004901 toroid\n  5 turns of RG174\n\nTransformer T2:\n  Fair-Rite 2843000202 core (BN-43-202)\n  0.3mm magnetic copper wire\n  1-2: 1 turn\n  2-3: 1 turn\n  4-5: 8 turns\n  6-7: 8 turns\n\nTransformer T3:\n  Fair-Rite 2843000202 core (BN-43-202)\n  10 turns of twisted pair made from\n  0.3mm magnetic copper wire\n
 Text Notes 4800 900  0    50   ~ 0
 Adjust response @ 20-30 MHz with C13.\nChange C10, C11 to 2.2 or 4.7pF if needed.
@@
 Wire Wire Line
 	3100 2350 3100 3000
+Text Notes 1600 900  0    50   ~ 0
+Transformers T1, T2, T3:\nsee TRANSFORMERS.md file for instructions
 $EndSCHEMATC
